File: electronics/eagle/project/measurementdevice.brd (EAGLE design)
At the start: 80 x 70 mm, 48 parts, among them U1 VX7805-1000, X1 MSTBA6

Commit message: [Electronics] First RC for circuit
Parts:
- removed C7, MD1:C5, MD2:C5, MD3:C5, MD4:C5: 0.1uF, rcl:C0805
- removed C8: 0.01uF, rcl:C0805
- removed L1: Ferrite Bead, rcl:L1812
- added LED2: GREEN, led:CHIP-LED0805
- added MD1:C6, MD2:C6, MD3:C6, MD4:C6: 1uF, rcl:C0603
- added MD1:C7, MD2:C7, MD3:C7, MD4:C7: 0.1uF, rcl:C0603
- added MD1:C8, MD2:C8, MD3:C8, MD4:C8: 0.01uF, rcl:C0603
- added MD1:L1, MD2:L1, MD3:L1, MD4:L1: Ferrite Bead, rcl:L1812
- added Q1: TN0604N3, transistor-fet:TO-92
- added R4: 1k, rcl:R0805
- added R5: 5, rcl:R1206
- added R6: 100, rcl:R0805
- C1: value 10uF -> 1uF
- C3: device rcl:C0805 -> rcl:C1206
- C4: value 22uF -> 10uF; device rcl:C0805 -> rcl:C1206
- C5: value 0.1uF -> 10uF; device rcl:C0805 -> rcl:C1206
- C6: value 1uF -> 0.1uF; device rcl:C0805 -> rcl:C1206
- D1: value 1N4004 -> 1N5819
- D2: value 1N5339B -> BZD23C5V6; device diode:C1702-15 -> diode:SOD81
- F1: value 2A -> 1.3A
- moved C1 401.4 mm to (27.0, 59.0), turned to 270 degrees
- moved C6 392.2 mm to (10.0, 48.0), turned to 180 degrees
- moved MD1:JP3 372.5 mm to (46.0, 58.0)
- moved MD2:JP3 368.0 mm to (46.0, 45.0)
- moved MD3:JP3 363.4 mm to (46.0, 32.0)
- moved MD4:JP3 358.9 mm to (46.0, 19.0)
- moved MD4:F1 337.0 mm to (60.0, 20.0)
- moved MD4:IC1 332.2 mm to (53.0, 17.0), turned to 270 degrees
- moved MD4:X1 322.3 mm to (76.0, 16.0), turned to 90 degrees
- moved MD4:R1 321.9 mm to (66.0, 13.0), turned to 90 degrees
- moved MD3:F1 316.9 mm to (60.0, 33.0)
- moved MD3:IC1 312.3 mm to (53.0, 30.0), turned to 270 degrees
- moved MD3:X1 303.4 mm to (76.0, 29.0), turned to 90 degrees
- moved MD3:R1 302.3 mm to (66.0, 26.0), turned to 90 degrees
- moved MD2:F1 297.4 mm to (60.0, 46.0)
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Connections:
- net MD1:N$1 renamed MD1:PWR_OUT
- net MD1:N$2 renamed MD1:PWR_IN
- net MD1:N$3 renamed MD1:SENSE1
- net MD1:N$4 renamed MD1:A0
- net MD1:N$5 renamed MD1:SENSE2
- net MD2:N$1 renamed MD2:PWR_OUT
- net MD2:N$2 renamed MD2:PWR_IN
- net MD2:N$3 renamed MD2:SENSE1
- net MD2:N$4 renamed MD2:A0
- net MD2:N$5 renamed MD2:SENSE2
- net MD3:N$1 renamed MD3:PWR_OUT
- net MD3:N$2 renamed MD3:PWR_IN
- net MD3:N$3 renamed MD3:SENSE1
- net MD3:N$4 renamed MD3:A0
- net MD3:N$5 renamed MD3:SENSE2
- net MD4:N$1 renamed MD4:PWR_OUT
- net MD4:N$2 renamed MD4:PWR_IN
- net MD4:N$3 renamed MD4:SENSE1
- net MD4:N$4 renamed MD4:A0
- net MD4:N$5 renamed MD4:SENSE2
- net N$7 renamed SDA
- net N$8 renamed SCL
- removed net 3V3_FILTERED: C6.2, C7.2, C8.2, L1.2, MD1:C5.1, MD1:IC1.6, MD1:JP3.2, MD2:C5.1, MD2:IC1.1, MD2:IC1.6, MD2:JP3.2, MD3:C5.1, MD3:IC1.6, MD3:JP3.2, MD4:C5.1, MD4:IC1.6, MD4:JP3.2, R2.2, R3.2
- new net MD1:3V3_FILTERED: MD1:C6.2, MD1:C7.2, MD1:C8.2, MD1:IC1.6, MD1:L1.2
- new net MD2:3V3_FILTERED: MD2:C6.2, MD2:C7.2, MD2:C8.2, MD2:IC1.6, MD2:L1.2
- new net MD3:3V3_FILTERED: MD3:C6.2, MD3:C7.2, MD3:C8.2, MD3:IC1.6, MD3:L1.2
- new net MD4:3V3_FILTERED: MD4:C6.2, MD4:C7.2, MD4:C8.2, MD4:IC1.6, MD4:L1.2
- new net N$10: Q1.1, R5.2
- new net N$5: D2.A, Q1.2, R4.2
- new net N$7: LED2.C, R6.2
- net +3V3: now also LED2.A, MD1:JP3.2, MD1:L1.1, MD2:IC1.1, MD2:JP3.2, MD2:L1.1, MD3:JP3.2, MD3:L1.1, MD4:JP3.2, MD4:L1.1, R2.2, R3.2; no longer L1.1
- net +5V: now also Q1.3
- net GND: now also C6.2, MD1:C6.1, MD1:C7.1, MD1:C8.1, MD2:C6.1, MD2:C7.1, MD2:C8.1, MD3:C6.1, MD3:C7.1, MD3:C8.1, MD4:C6.1, MD4:C7.1, MD4:C8.1, R4.1, R5.1, R6.1; no longer C6.1, C7.1, C8.1, D2.A, MD1:C5.2, MD2:C5.2, MD3:C5.2, MD4:C5.2
- net N$9: now also C6.1
Routing:
- net SCL: track 0.00 -> 183.6 mm, vias 0 -> 4
- net +3V3: track 0.00 -> 168.6 mm, vias 0 -> 6
- net SDA: track 0.00 -> 144.6 mm
- net PB11: track 0.00 -> 105.3 mm
- net PB10: track 0.00 -> 36.6 mm
- net 3V3: track 0.00 -> 23.7 mm
- net N$6: track 31.3 -> 11.7 mm
- net GND: track 16.1 -> 0.00 mm, vias 4 -> 37
- net N$9: track 0.00 -> 14.5 mm
- net N$2: track 16.4 -> 3.49 mm
- net MD4:A0: track 0.00 -> 12.3 mm
- net MD3:A0: track 0.00 -> 12.3 mm
- net MD2:A0: track 0.00 -> 12.3 mm
- net MD1:A0: track 0.00 -> 12.3 mm
- net MD3:3V3_FILTERED: track 0.00 -> 12.2 mm
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- added copper zone on layer 1, net GND
- added copper zone on layer 1, net MD1:PWR_IN
- added copper zone on layer 1, net MD1:PWR_OUT
- added copper zone on layer 1, net MD2:PWR_IN
- added copper zone on layer 1, net MD2:PWR_OUT
- added copper zone on layer 1, net MD3:PWR_IN
- added copper zone on layer 1, net MD3:PWR_OUT
- added copper zone on layer 1, net MD4:PWR_IN
- added copper zone on layer 1, net MD4:PWR_OUT

Commit message: [Electronics] Last version
Parts:
- added X2: PT1.5/3-50H-3, PersonalLibrary:PT1.5/3-50H-3
- C1: device rcl:C0805 -> rcl:C0603
- C6: device rcl:C1206 -> rcl:C0603
- D2: device diode:SOD81 -> PersonalLibrary:SOD81-ED
- F1: device fuse:LITTLEFUSE -> PersonalLibrary:LITTLEFUSE
- MD1:F1, MD2:F1, MD3:F1, MD4:F1: device PersonalLibrary:16R1000G -> PersonalLibrary:RUEF900
- MD1:L1, MD2:L1, MD3:L1, MD4:L1: device rcl:L1812 -> PersonalLibrary:0603
- MD1:X1, MD2:X1, MD3:X1, MD4:X1: value MSTBA2 -> PT1.5/3-50H-2; device con-phoenix-508:MSTBA2 -> PersonalLibrary:PT1.5/3-50H-2
- R1: value 560 -> 240
- X1: value MSTBA6 -> PT1.5/3-50H-3; device con-phoenix-508:MSTBA6 -> PersonalLibrary:PT1.5/3-50H-3
- moved C1 15.2 mm to (24.5, 44.0), turned to 0 degrees
- moved MD4:F1 14.6 mm to (45.5, 18.0)
- moved MD3:F1 14.6 mm to (45.5, 31.5)
- moved MD2:F1 14.5 mm to (45.5, 45.0)
- moved MD1:F1 14.5 mm to (45.5, 58.5)
- moved C6 14.0 mm to (24.0, 48.0), turned to 0 degrees
- moved R5 10.1 mm to (22.5, 25.0), turned to 0 degrees
- moved MD4:L1 8.73 mm to (55.5, 10.0)
- moved MD3:L1 8.63 mm to (55.5, 23.5)
- moved MD2:L1 8.51 mm to (55.5, 37.5)
- moved MD1:L1 8.50 mm to (55.5, 51.0)
- moved MD1:X1 8.14 mm to (70.5, 61.0), turned to 270 degrees
- moved MD2:X1 7.78 mm to (70.5, 47.5), turned to 270 degrees
- moved MD3:X1 7.43 mm to (70.5, 34.0), turned to 270 degrees
- moved MD4:X1 7.11 mm to (70.5, 20.5), turned to 270 degrees
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Connections:
- removed net MD2:3V3_FILTERED: MD2:C6.2, MD2:C7.2, MD2:C8.2, MD2:IC1.6, MD2:L1.2
- new net N$8: Q1.3, R5.1
- net +3V3: now also MD1:C6.2, MD1:L1.N1, MD2:C6.2, MD2:L1.N1, MD3:C6.2, MD3:L1.N1, MD4:C6.2, MD4:L1.N1; no longer MD1:JP3.2, MD1:L1.1, MD2:IC1.1, MD2:JP3.2, MD2:L1.1, MD3:JP3.2, MD3:L1.1, MD4:JP3.2, MD4:L1.1
- net +5V: now also R5.2; no longer Q1.3
- net GND: now also MD1:X1.P$1, MD2:X1.P$1, MD3:X1.P$1, MD4:X1.P$1, Q1.1, X2.P$1, X2.P$2, X2.P$3; no longer MD1:X1.2, MD2:X1.2, MD3:X1.2, MD4:X1.2, R5.1, X1.4, X1.5, X1.6
- net MD1:3V3_FILTERED: now also MD1:JP3.2, MD1:L1.N2; no longer MD1:C6.2, MD1:L1.2
- net MD1:PWR_OUT: now also MD1:X1.P$2; no longer MD1:X1.1
- net MD2:PWR_OUT: now also MD2:X1.P$2; no longer MD2:X1.1
- net MD3:3V3_FILTERED: now also MD3:JP3.2, MD3:L1.N2; no longer MD3:C6.2, MD3:L1.2
- net MD3:PWR_OUT: now also MD3:X1.P$2; no longer MD3:X1.1
- net MD4:3V3_FILTERED: now also MD4:JP3.2, MD4:L1.N2; no longer MD4:C6.2, MD4:L1.2
- net MD4:PWR_OUT: now also MD4:X1.P$2; no longer MD4:X1.1
- net N$10: now also MD2:C7.2, MD2:C8.2, MD2:IC1.1, MD2:IC1.6, MD2:JP3.2, MD2:L1.N2; no longer Q1.1, R5.2
- net V+: now also X1.P$1, X1.P$2, X1.P$3; no longer X1.1, X1.2, X1.3
Routing:
- net SCL: track 183.6 -> 127.0 mm, vias 4 -> 0
- net GND: track 0.00 -> 37.9 mm, vias 37 -> 42
- net SDA: track 144.6 -> 116.5 mm
- net N$10: track 3.31 -> 25.8 mm
- net MD1:3V3_FILTERED: track 12.1 -> 29.7 mm
- net MD4:3V3_FILTERED: track 12.1 -> 26.3 mm
- net MD3:3V3_FILTERED: track 12.2 -> 26.3 mm
- net PB11: track 105.3 -> 117.6 mm, vias 0 -> 1
- net MD2:3V3_FILTERED: track 12.1 -> 0.00 mm
- net +3V3: track 168.6 -> 160.9 mm
- net MD1:A0: track 12.3 -> 18.0 mm, vias 0 -> 1
- net MD4:SENSE1: track 4.50 -> 8.91 mm
- net N$5: track 9.33 -> 13.3 mm
- net N$9: track 14.5 -> 10.5 mm
- net MD3:SENSE1: track 4.44 -> 8.36 mm
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Other:
- board text added: "3V3"
- board text added: "5V"
- board text added: "AP"
- board text added: "C6"
- board text added: "C7"
- board text added: "C8"
- board text added: "Designed by F.Reghenzani"
- board text added: "GND"
- board text added: "HE"
- board text added: "IC1"
- board text added: "IF = 5V"
- board text added: "IF > 5V"
- board text added: "L1"
- board text added: "Lab"
- board text added: "Politecnico"
- board text added: "R1"
- board text added: "SmokyProbe"
- board text added: "V+"
- board text added: "Zaneeeeeeeeella"
- board text added: "di Milano"
- board text added: "v1.0"
- board text added: "v1.0 2019"
