File: electronics/eagle/project/measurementdevice.sch (EAGLE design)
At the start: 24 parts, among them U1 VX7805-1000, X1 MSTBA6

Commit message: [Electronics] First RC for circuit
Parts:
- removed C7: 0.1uF, rcl:C-EUC0805
- removed C8: 0.01uF, rcl:C-EUC0805
- removed L1: Ferrite Bead, rcl:L-USL1812
- added LED2: GREEN, led:LEDCHIP-LED0805
- added Q1: TN0604N3, transistor-fet:TN0604N3
- added R4: 1k, rcl:R-EU_R0805
- added R5: 5, rcl:R-EU_R1206
- added R6: 100, rcl:R-EU_R0805
- C1: value 10uF -> 1uF
- C3: device rcl:C-EUC0805 -> rcl:C-EUC1206
- C4: value 22uF -> 10uF; device rcl:C-EUC0805 -> rcl:C-EUC1206
- C5: value 0.1uF -> 10uF; device rcl:C-EUC0805 -> rcl:C-EUC1206
- C6: value 1uF -> 0.1uF; device rcl:C-EUC0805 -> rcl:C-EUC1206
- D1: value 1N4004 -> 1N5819; device diode:1N4004 -> diode:1N4933
- D2: value 1N5339B -> BZD23C5V6; device diode:1N5333 -> diode:BZD23
- F1: value 2A -> 1.3A
Connections:
- net N$5 renamed SENSE2
- removed net N$8: JP3.6, JP3.8, R2.1
- new net A0: JP3.1, JP3.3, JP3.5, JP3.7
- new net N$10: Q1.S, R5.2
- new net N$5: D2.A, Q1.G, R4.2
- new net PWR_IN: F1.P$2, R1.I2
- new net PWR_OUT: R1.I1, X1-1.1
- new net SENSE1: R1.V2
- net +3V3: now also LED2.A, R2.2, R3.2; no longer C5.1, L1.1
- net +5V: now also Q1.D
- net 3V3_FILTERED: no longer C7.2, C8.2, L1.2, R2.2, R3.2
- net GND: now also C6.2, R4.1, R5.1, R6.1; no longer C7.1, C8.1, D2.A
- net N$1: no longer R1.I1, X1-1.1
- net N$2: no longer F1.P$2, R1.I2
- net N$3: no longer R1.V2
- net N$4: no longer JP3.1, JP3.3, JP3.5, JP3.7
- net N$7: now also LED2.C, R6.2; no longer JP3.2, JP3.4, R3.1
- net N$9: now also C6.1
- net SCL: now also JP3.8, R2.1
- net SDA: now also JP3.2, R3.1
Other:
- note added: "Over-voltage and over-current protection"
- note removed: "Protection diode"
- moved on the sheet: C5, D2, F1, LED1, R1

Commit message: [Electronics] Last version
Parts:
- added X2: PT1.5/3-50H-3, PersonalLibrary:PT1.5/3-50H-3
- C1: device rcl:C-EUC0805 -> rcl:C-EUC0603
- C6: device rcl:C-EUC1206 -> rcl:C-EUC0603
- D2: device diode:BZD23 -> PersonalLibrary:1N5339BG
- F1: device fuse:LITTLEFUSE -> PersonalLibrary:LITTLEFUSE; SPICEPREFIX (none) -> F
- R1: value 560 -> 240
- X1: value MSTBA6 -> PT1.5/3-50H-3; device con-phoenix-508:MSTBA6 -> PersonalLibrary:PT1.5/3-50H-3
Connections:
- removed net N$10: Q1.S, R5.2
- new net N$8: Q1.D, R5.1
- net +3V3: now also C6.2; no longer JP3.2
- net +5V: now also R5.2; no longer Q1.D
- net 3V3_FILTERED: now also JP3.2; no longer C6.2
- net GND: now also Q1.S, X1G$1.SK, X2G$1.SK, X2G$2.SK, X2G$3.SK; no longer R5.1, X1-2.1, X1-4.1, X1-5.1, X1-6.1
- net PWR_OUT: now also X1G$2.SK; no longer X1-1.1
- net V+: now also X1G$1.SK, X1G$2.SK, X1G$3.SK; no longer X1-1.1, X1-2.1, X1-3.1
